Commit message: add send destination to server

File: src/roscar_description/urdf/roscar.urdf.xacro (robot description, xacro)
@@ -9,4 +9,8 @@
   <xacro:arg name="imu_z" default="0.0"/>
   <xacro:arg name="imu_yaw" default="0.0"/>
+  <xacro:arg name="camera_x" default="0.0"/>
+  <xacro:arg name="camera_y" default="0.0"/>
+  <xacro:arg name="camera_z" default="0.20"/>
+  <xacro:arg name="camera_yaw" default="0.0"/>
   <link name="base_footprint"/>
   <link name="base_link">
@@ -36,3 +40,11 @@
     <parent link="base_link"/><child link="imu_link"/>
   </joint>
+  <!-- r200_link 之下的光学系(r200_*_optical_frame)由 r200_node 从 SDK 外参发布,
+       不写入 URDF。 -->
+  <link name="r200_link"/>
+  <joint name="r200_joint" type="fixed">
+    <origin xyz="$(arg camera_x) $(arg camera_y) $(arg camera_z)"
+            rpy="0 0 $(arg camera_yaw)"/>
+    <parent link="base_link"/><child link="r200_link"/>
+  </joint>
 </robot>
